Commit message: Adição link_1.stl e link_2.stl

File: install/6dof_arm_description/share/6dof_arm_description/urdf/6dof_arm.urdf.xacro (robot description, xacro)
@@ -1,4 +1 @@
-<?xml version="1.0"?>
-<robot name="6dof_arm" xmlns:xacro="http://www.ros.org/wiki/xacro">
-    <xacro:include filename="mobile_base.xacro"/>
-</robot>
+/home/livia/rl_6dof_ws/src/6dof_arm_description/urdf/6dof_arm.urdf.xacro

File: install/6dof_arm_description/share/6dof_arm_description/urdf/mobile_base.xacro (robot description, xacro)
@@ -1,20 +1 @@
-<?xml version="1.0"?>
-<robot xmlns:xacro="http://www.ros.org/wiki/xacro">
-    <material name="light_black">
-        <color rgba="0.4 0.4 0.4 1.0"/>
-    </material>
-    <link name="base_footprint"/>
-    <link name="base_link">
-        <visual>
-            <geometry>
-                <mesh filename="package://6dof_arm_description/meshes/6dof_arm/base_link.stl" scale="1 1 1"/>
-            </geometry>
-            <material name="light_black"/>
-        </visual>
-    </link>
-    <joint name="base_joint" type="fixed">
-        <parent link="base_footprint" />
-        <child link="base_link" />
-        <origin xyz ="0 0 0" rpy="0 0 0" />
-    </joint>
-</robot>
+/home/livia/rl_6dof_ws/src/6dof_arm_description/urdf/mobile_base.xacro

File: src/6dof_arm_description/urdf/mobile_base.xacro (robot description, xacro)
@@ -8,6 +8,25 @@
         <visual>
             <geometry>
-                <mesh filename="package://6dof_arm_description/meshes/6dof_arm/base_link.stl" scale="1 1 1"/>
+                <mesh filename="package://6dof_arm_description/meshes/6dof_arm/base_link.stl"/>
             </geometry>
+            <origin xyz="0 0 0.04" rpy="0 0 0"/>
+            <material name="light_black"/>
+        </visual>
+    </link>
+    <link name="arm_1_link">
+        <visual>
+            <geometry>
+                <mesh filename="package://6dof_arm_description/meshes/6dof_arm/link_1.stl"/>
+            </geometry>
+            <origin xyz="0 0 0.07" rpy="0 0 0"/>
+            <material name="light_black"/>
+        </visual>
+    </link>
+    <link name="arm_2_link">
+        <visual>
+            <geometry>
+                <mesh filename="package://6dof_arm_description/meshes/6dof_arm/link_2.stl"/>
+            </geometry>
+            <origin xyz="0 0.15 0" rpy="0 0 ${pi/2.0}"/>
             <material name="light_black"/>
         </visual>
@@ -18,3 +37,15 @@
         <origin xyz ="0 0 0" rpy="0 0 0" />
     </joint>
+    <joint name="base_arm_1_joint" type="continuous">
+        <parent link="base_link" />
+        <child link="arm_1_link" />
+        <origin xyz ="0 0 0" rpy="0 0 0" />
+        <axis xyz="0 0 1" />
+    </joint>
+    <joint name="base_arm_2_joint" type="continuous">
+        <parent link="arm_1_link" />
+        <child link="arm_2_link" />
+        <origin xyz ="0 0 0.27" rpy="0 0 0" />
+        <axis xyz="0 1 0" />
+    </joint>
 </robot>
