Commit message: Adição de colisão

File: src/6dof_arm_description/urdf/mobile_base.xacro (robot description, xacro)
@@ -10,4 +10,10 @@
             <material name="light_black"/>
         </visual>
+        <collision>
+            <geometry>
+                <cylinder radius="0.15" length="0.07" />
+            </geometry>
+            <origin xyz="0 0 0.035" rpy="0 0 0"/>
+        </collision>
         <xacro:base_link xyz="0 2.679e-8 0.01026544" rpy="0 0 0" />
     </link>
@@ -20,4 +26,10 @@
             <material name="salmon"/>
         </visual>
+        <collision>
+            <geometry>
+                <box size="0.15 0.20 0.275" />
+            </geometry>
+            <origin xyz="0 0 0.1375" rpy="0 0 0"/>
+        </collision>
         <xacro:arm1_link xyz="0 -0.00016159 0.14671717" rpy="0 0 0" />
     </link>
@@ -30,4 +42,10 @@
             <material name="yellow"/>
         </visual>
+        <collision>
+            <geometry>
+                <box size="0.15 0.20 1.10" />
+            </geometry>
+            <origin xyz="0 0 0.475" rpy="0 0 0"/>
+        </collision>
         <xacro:arm2_link xyz="-0.00008884 0 0.47500021" rpy="0 0 -${pi/2.0}" />
     </link>
@@ -40,4 +58,10 @@
             <material name="purple"/>
         </visual>
+        <collision>
+            <geometry>
+                <box size="0.15 0.20 0.80" />
+            </geometry>
+            <origin xyz="0.325 0 0" rpy="0 ${pi/2} 0"/>
+        </collision>
         <xacro:arm3_link xyz="0.325 0 -0.00011793" rpy="0 ${pi/2} 0" />
     </link>
@@ -50,4 +74,10 @@
             <material name="green"/>
         </visual>
+        <collision>
+            <geometry>
+                <box size="0.15 0.20 0.275" />
+            </geometry>
+            <origin xyz="0 0 -0.0625" rpy="0 0 0"/>
+        </collision>
         <xacro:arm4_link xyz="0 0.0010614 -0.05328286" rpy="${pi} 0 0" />
     </link>
@@ -60,4 +90,10 @@
             <material name="blue"/>
         </visual>
+        <collision>
+            <geometry>
+                <box size="0.20 0.15 0.175" />
+            </geometry>
+            <origin xyz="0 0 -0.0875" rpy="0 0 0"/>
+        </collision>
         <xacro:arm5_link xyz="-0.0002301 0 -0.08772699" rpy="${pi} 0 ${pi}" />
     </link>
@@ -70,4 +106,10 @@
             <material name="blue_tifany"/>
         </visual>
+        <collision>
+            <geometry>
+                <box size="0.15 0.15 0.20" />
+            </geometry>
+            <origin xyz="0 0 0.10" rpy="0 0 0"/>
+        </collision>
         <xacro:arm6_link xyz="0 0 0.10531595" rpy="0 0 0" />
     </link>
