Commit message: Adição link_3.stl, link_4.stl, link_5.stl e link_6.stl

File: src/6dof_arm_description/urdf/6dof_arm.urdf.xacro (robot description, xacro)
@@ -2,3 +2,4 @@
 <robot name="6dof_arm" xmlns:xacro="http://www.ros.org/wiki/xacro">
     <xacro:include filename="mobile_base.xacro"/>
+    <xacro:include filename="properties.urdf.xacro"/>
 </robot>

File: src/6dof_arm_description/urdf/mobile_base.xacro (robot description, xacro)
@@ -1,12 +1,9 @@
 <?xml version="1.0"?>
 <robot xmlns:xacro="http://www.ros.org/wiki/xacro">
-    <material name="light_black">
-        <color rgba="0.4 0.4 0.4 1.0"/>
-    </material>
     <link name="base_footprint"/>
     <link name="base_link">
         <visual>
             <geometry>
-                <mesh filename="package://6dof_arm_description/meshes/6dof_arm/base_link.stl"/>
+                <mesh filename="package://6dof_arm_description/meshes/6dof_arm/base_link.stl" scale="1 1 1"/>
             </geometry>
             <origin xyz="0 0 0.04" rpy="0 0 0"/>
@@ -17,8 +14,8 @@
         <visual>
             <geometry>
-                <mesh filename="package://6dof_arm_description/meshes/6dof_arm/link_1.stl"/>
+                <mesh filename="package://6dof_arm_description/meshes/6dof_arm/link_1.stl" scale="1 1 1"/>
             </geometry>
-            <origin xyz="0 0 0.07" rpy="0 0 0"/>
-            <material name="light_black"/>
+            <origin xyz="0 0 0" rpy="0 0 0"/>
+            <material name="salmon"/>
         </visual>
     </link>
@@ -26,8 +23,44 @@
         <visual>
             <geometry>
-                <mesh filename="package://6dof_arm_description/meshes/6dof_arm/link_2.stl"/>
+                <mesh filename="package://6dof_arm_description/meshes/6dof_arm/link_2.stl" scale="1 1 1"/>
             </geometry>
-            <origin xyz="0 0.15 0" rpy="0 0 ${pi/2.0}"/>
-            <material name="light_black"/>
+            <origin xyz="0 0 0" rpy="0 0 -${pi/2.0}"/>
+            <material name="yellow"/>
+        </visual>
+    </link>
+    <link name="arm_3_link">
+        <visual>
+            <geometry>
+                <mesh filename="package://6dof_arm_description/meshes/6dof_arm/link_3.stl" scale="1 1 1"/>
+            </geometry>
+            <origin xyz="0 0 0" rpy="0 ${pi/2} 0"/>
+            <material name="purple"/>
+        </visual>
+    </link>
+    <link name="arm_4_link">
+        <visual>
+            <geometry>
+                <mesh filename="package://6dof_arm_description/meshes/6dof_arm/link_4.stl" scale="1 1 1"/>
+            </geometry>
+            <origin xyz="0 0 0" rpy="${pi} 0 0"/>
+            <material name="green"/>
+        </visual>
+    </link>
+    <link name="arm_5_link">
+        <visual>
+            <geometry>
+                <mesh filename="package://6dof_arm_description/meshes/6dof_arm/link_5.stl" scale="1 1 1"/>
+            </geometry>
+            <origin xyz="0 0 0" rpy="${pi} 0 ${pi}"/>
+            <material name="blue"/>
+        </visual>
+    </link>
+    <link name="arm_6_link">
+        <visual>
+            <geometry>
+                <mesh filename="package://6dof_arm_description/meshes/6dof_arm/link_6.stl" scale="1 1 1"/>
+            </geometry>
+            <origin xyz="0 0 0" rpy="0 0 0"/>
+            <material name="blue_tifany"/>
         </visual>
     </link>
@@ -40,12 +73,36 @@
         <parent link="base_link" />
         <child link="arm_1_link" />
-        <origin xyz ="0 0 0" rpy="0 0 0" />
+        <origin xyz ="0 0 0.07" rpy="0 0 0" />
         <axis xyz="0 0 1" />
     </joint>
-    <joint name="base_arm_2_joint" type="continuous">
+    <joint name="arm_1_arm_2_joint" type="continuous">
         <parent link="arm_1_link" />
         <child link="arm_2_link" />
-        <origin xyz ="0 0 0.27" rpy="0 0 0" />
+        <origin xyz ="0 -0.20 0.20" rpy="0 0 0" />
         <axis xyz="0 1 0" />
     </joint>
+    <joint name="arm_2_arm_3_joint" type="continuous">
+        <parent link="arm_2_link" />
+        <child link="arm_3_link" />
+        <origin xyz ="0 0.20 0.95" rpy="0 0 0" />
+        <axis xyz="0 1 0" />
+    </joint>
+    <joint name="arm_3_arm_4_joint" type="continuous">
+        <parent link="arm_3_link" />
+        <child link="arm_4_link" />
+        <origin xyz ="0.65 -0.20 0" rpy="0 -${pi/2} 0" />
+        <axis xyz="0 1 0" />
+    </joint>
+    <joint name="arm_4_arm_5_joint" type="continuous">
+        <parent link="arm_4_link" />
+        <child link="arm_5_link" />
+        <origin xyz ="0 0 -0.20" rpy="0 0 ${pi}" />
+        <axis xyz="0 0 1" />
+    </joint>
+    <joint name="arm_5_arm_6_joint" type="continuous">
+        <parent link="arm_5_link" />
+        <child link="arm_6_link" />
+        <origin xyz ="0.10 0 -0.1" rpy="0 ${pi/2} 0" />
+        <axis xyz="0 0 1" />
+    </joint>
 </robot>

Commit message: Adição de momentos de inércia

File: src/6dof_arm_description/urdf/6dof_arm.urdf.xacro (robot description, xacro)
@@ -1,5 +1,5 @@
 <?xml version="1.0"?>
 <robot name="6dof_arm" xmlns:xacro="http://www.ros.org/wiki/xacro">
+    <xacro:include filename="properties.urdf.xacro"/>
     <xacro:include filename="mobile_base.xacro"/>
-    <xacro:include filename="properties.urdf.xacro"/>
 </robot>

File: src/6dof_arm_description/urdf/mobile_base.xacro (robot description, xacro)
@@ -10,6 +10,7 @@
             <material name="light_black"/>
         </visual>
+        <xacro:base_link xyz="0 2.679e-8 0.01026544" rpy="0 0 0" />
     </link>
-    <link name="arm_1_link">
+    <link name="arm1_link">
         <visual>
             <geometry>
@@ -19,6 +20,7 @@
             <material name="salmon"/>
         </visual>
+        <xacro:arm1_link xyz="0 -0.00016159 0.14671717" rpy="0 0 0" />
     </link>
-    <link name="arm_2_link">
+    <link name="arm2_link">
         <visual>
             <geometry>
@@ -28,6 +30,7 @@
             <material name="yellow"/>
         </visual>
+        <xacro:arm2_link xyz="-0.00008884 0 0.47500021" rpy="0 0 -${pi/2.0}" />
     </link>
-    <link name="arm_3_link">
+    <link name="arm3_link">
         <visual>
             <geometry>
@@ -37,6 +40,7 @@
             <material name="purple"/>
         </visual>
+        <xacro:arm3_link xyz="0.325 0 -0.00011793" rpy="0 ${pi/2} 0" />
     </link>
-    <link name="arm_4_link">
+    <link name="arm4_link">
         <visual>
             <geometry>
@@ -46,6 +50,7 @@
             <material name="green"/>
         </visual>
+        <xacro:arm4_link xyz="0 0.0010614 -0.05328286" rpy="${pi} 0 0" />
     </link>
-    <link name="arm_5_link">
+    <link name="arm5_link">
         <visual>
             <geometry>
@@ -55,6 +60,7 @@
             <material name="blue"/>
         </visual>
+        <xacro:arm5_link xyz="-0.0002301 0 -0.08772699" rpy="${pi} 0 ${pi}" />
     </link>
-    <link name="arm_6_link">
+    <link name="arm6_link">
         <visual>
             <geometry>
@@ -64,4 +70,5 @@
             <material name="blue_tifany"/>
         </visual>
+        <xacro:arm6_link xyz="0 0 0.10531595" rpy="0 0 0" />
     </link>
     <joint name="base_joint" type="fixed">
@@ -70,37 +77,37 @@
         <origin xyz ="0 0 0" rpy="0 0 0" />
     </joint>
-    <joint name="base_arm_1_joint" type="continuous">
+    <joint name="base_arm1_joint" type="continuous">
         <parent link="base_link" />
-        <child link="arm_1_link" />
+        <child link="arm1_link" />
         <origin xyz ="0 0 0.07" rpy="0 0 0" />
         <axis xyz="0 0 1" />
     </joint>
-    <joint name="arm_1_arm_2_joint" type="continuous">
-        <parent link="arm_1_link" />
-        <child link="arm_2_link" />
+    <joint name="arm1_arm2_joint" type="continuous">
+        <parent link="arm1_link" />
+        <child link="arm2_link" />
         <origin xyz ="0 -0.20 0.20" rpy="0 0 0" />
         <axis xyz="0 1 0" />
     </joint>
-    <joint name="arm_2_arm_3_joint" type="continuous">
-        <parent link="arm_2_link" />
-        <child link="arm_3_link" />
+    <joint name="arm2_arm3_joint" type="continuous">
+        <parent link="arm2_link" />
+        <child link="arm3_link" />
         <origin xyz ="0 0.20 0.95" rpy="0 0 0" />
         <axis xyz="0 1 0" />
     </joint>
-    <joint name="arm_3_arm_4_joint" type="continuous">
-        <parent link="arm_3_link" />
-        <child link="arm_4_link" />
+    <joint name="arm3_arm4_joint" type="continuous">
+        <parent link="arm3_link" />
+        <child link="arm4_link" />
         <origin xyz ="0.65 -0.20 0" rpy="0 -${pi/2} 0" />
         <axis xyz="0 1 0" />
     </joint>
-    <joint name="arm_4_arm_5_joint" type="continuous">
-        <parent link="arm_4_link" />
-        <child link="arm_5_link" />
+    <joint name="arm4_arm5_joint" type="continuous">
+        <parent link="arm4_link" />
+        <child link="arm5_link" />
         <origin xyz ="0 0 -0.20" rpy="0 0 ${pi}" />
         <axis xyz="0 0 1" />
     </joint>
-    <joint name="arm_5_arm_6_joint" type="continuous">
-        <parent link="arm_5_link" />
-        <child link="arm_6_link" />
+    <joint name="arm5_arm6_joint" type="continuous">
+        <parent link="arm5_link" />
+        <child link="arm6_link" />
         <origin xyz ="0.10 0 -0.1" rpy="0 ${pi/2} 0" />
         <axis xyz="0 0 1" />

File: src/6dof_arm_description/urdf/properties.urdf.xacro (robot description, xacro)
@@ -22,29 +22,65 @@
         <color rgba="0.5372 0.8549 0.8274 1.0"/>
     </material>
-    <xacro:macro name="box_inertia" params="m l w h xyz rpy">
+    <xacro:macro name="base_link" params="xyz rpy">
         <inertial>
             <origin xyz="${xyz}" rpy="${rpy}" />
-            <mass value="${m}" />
-            <inertia ixx="${(m/12) * (h*h + l*l)}" ixy="0" ixz="0"
-                     iyy="${(m/12) * (w*w + l*l)}"  iyz="0"
-                     izz="${(m/12) * (w*w + h*h)}" />
+            <mass value="10.6734184" />
+            <inertia ixx="0.05702778" ixy="0" ixz="0"
+                     iyy="0.05702779"  iyz="0"
+                     izz="0.10703462" />
         </inertial>
     </xacro:macro>
-    <xacro:macro name="wheel_inertia" params="m r h xyz rpy">
+    <xacro:macro name="arm1_link" params="xyz rpy">
         <inertial>
             <origin xyz="${xyz}" rpy="${rpy}" />
-            <mass value="${m}" />
-            <inertia ixx="${(m/12) * (3*r*r + h*h)}" ixy="0" ixz="0"
-                     iyy="${(m/12) * (3*r*r + h*h)}"  iyz="0"
-                     izz="${(1/2) * (m * r*r)}" />
+            <mass value="16.02392927" />
+            <inertia ixx="0.13097774" ixy="-1.354e-8" ixz="0"
+                     iyy="0.11390137"  iyz="0.00013796"
+                     izz="0.06378491" />
         </inertial>
     </xacro:macro>
-    <xacro:macro name="caster_wheel_inertia" params="m r xyz rpy">
+    <xacro:macro name="arm2_link" params="xyz rpy">
         <inertial>
             <origin xyz="${xyz}" rpy="${rpy}" />
-            <mass value="${m}" />
-            <inertia ixx="${(2/5) * (m*r*r)}" ixy="0" ixz="0"
-                     iyy="${(2/5) * (m*r*r)}"  iyz="0"
-                     izz="${(2/5) * (m*r*r)}" />
+            <mass value="58.29018559" />
+            <inertia ixx="6.62579145" ixy="0.0000054" ixz="0"
+                     iyy="6.65994246"  iyz="-4e-8"
+                     izz="0.20137485" />
+        </inertial>
+    </xacro:macro>
+    <xacro:macro name="arm3_link" params="xyz rpy">
+        <inertial>
+            <origin xyz="${xyz}" rpy="${rpy}" />
+            <mass value="43.97624328" />
+            <inertia ixx="0.16111702" ixy="0" ixz="-9.935e-8"
+                     iyy="2.67279881"  iyz="5.713e-9"
+                     izz="2.70695549" />
+        </inertial>
+    </xacro:macro>
+    <xacro:macro name="arm4_link" params="xyz rpy">
+        <inertial>
+            <origin xyz="${xyz}" rpy="${rpy}" />
+            <mass value="16.02394366" />
+            <inertia ixx="0.13101946" ixy="1.335e-8" ixz="-2.826e-9"
+                     iyy="0.11390118"  iyz="-0.00166483"
+                     izz="0.06382633" />
+        </inertial>
+    </xacro:macro>
+    <xacro:macro name="arm5_link" params="xyz rpy">
+        <inertial>
+            <origin xyz="${xyz}" rpy="${rpy}" />
+            <mass value="11.25261767" />
+            <inertia ixx="0.03965941" ixy="2.335e-9" ixz="0.00003178"
+                     iyy="0.05673546"  iyz="-6.760e-10"
+                     izz="0.05036553" />
+        </inertial>
+    </xacro:macro>
+    <xacro:macro name="arm6_link" params="xyz rpy">
+        <inertial>
+            <origin xyz="${xyz}" rpy="${rpy}" />
+            <mass value="9.94813346" />
+            <inertia ixx="0.05211159" ixy="0" ixz="0"
+                     iyy="0.05197757"  iyz="0"
+                     izz="0.02702159" />
         </inertial>
     </xacro:macro>

Commit message: Implementação de launch para o gazebo

File: src/6dof_arm_description/urdf/6dof_arm.urdf.xacro (robot description, xacro)
@@ -2,4 +2,4 @@
 <robot name="6dof_arm" xmlns:xacro="http://www.ros.org/wiki/xacro">
     <xacro:include filename="properties.urdf.xacro"/>
-    <xacro:include filename="mobile_base.xacro"/>
+    <xacro:include filename="mobile_base.urdf.xacro"/>
 </robot>

File: src/6dof_arm_description/urdf/mobile_base.urdf.xacro (robot description, xacro)
@@ -10,4 +10,5 @@
             <material name="light_black"/>
         </visual>
+        <xacro:base_inertia xyz="0 2.679e-8 0.01026544" rpy="0 0 0" />
         <collision>
             <geometry>
@@ -16,5 +17,4 @@
             <origin xyz="0 0 0.035" rpy="0 0 0"/>
         </collision>
-        <xacro:base_link xyz="0 2.679e-8 0.01026544" rpy="0 0 0" />
     </link>
     <link name="arm1_link">
@@ -26,4 +26,5 @@
             <material name="salmon"/>
         </visual>
+        <xacro:arm1_inertia xyz="0 -0.00016159 0.14671717" rpy="0 0 0" />
         <collision>
             <geometry>
@@ -32,5 +33,4 @@
             <origin xyz="0 0 0.1375" rpy="0 0 0"/>
         </collision>
-        <xacro:arm1_link xyz="0 -0.00016159 0.14671717" rpy="0 0 0" />
     </link>
     <link name="arm2_link">
@@ -42,4 +42,5 @@
             <material name="yellow"/>
         </visual>
+        <xacro:arm2_inertia xyz="-0.00008884 0 0.47500021" rpy="0 0 -${pi/2.0}" />
         <collision>
             <geometry>
@@ -48,5 +49,4 @@
             <origin xyz="0 0 0.475" rpy="0 0 0"/>
         </collision>
-        <xacro:arm2_link xyz="-0.00008884 0 0.47500021" rpy="0 0 -${pi/2.0}" />
     </link>
     <link name="arm3_link">
@@ -58,4 +58,5 @@
             <material name="purple"/>
         </visual>
+        <xacro:arm3_inertia xyz="0.325 0 -0.00011793" rpy="0 ${pi/2} 0" />
         <collision>
             <geometry>
@@ -64,5 +65,4 @@
             <origin xyz="0.325 0 0" rpy="0 ${pi/2} 0"/>
         </collision>
-        <xacro:arm3_link xyz="0.325 0 -0.00011793" rpy="0 ${pi/2} 0" />
     </link>
     <link name="arm4_link">
@@ -74,4 +74,5 @@
             <material name="green"/>
         </visual>
+        <xacro:arm4_inertia xyz="0 0.0010614 -0.05328286" rpy="${pi} 0 0" />
         <collision>
             <geometry>
@@ -80,5 +81,4 @@
             <origin xyz="0 0 -0.0625" rpy="0 0 0"/>
         </collision>
-        <xacro:arm4_link xyz="0 0.0010614 -0.05328286" rpy="${pi} 0 0" />
     </link>
     <link name="arm5_link">
@@ -90,4 +90,5 @@
             <material name="blue"/>
         </visual>
+        <xacro:arm5_inertia xyz="-0.0002301 0 -0.08772699" rpy="${pi} 0 ${pi}" />
         <collision>
             <geometry>
@@ -96,5 +97,4 @@
             <origin xyz="0 0 -0.0875" rpy="0 0 0"/>
         </collision>
-        <xacro:arm5_link xyz="-0.0002301 0 -0.08772699" rpy="${pi} 0 ${pi}" />
     </link>
     <link name="arm6_link">
@@ -106,4 +106,5 @@
             <material name="blue_tifany"/>
         </visual>
+        <xacro:arm6_inertia xyz="0 0 0.10531595" rpy="0 0 0" />
         <collision>
             <geometry>
@@ -112,5 +113,4 @@
             <origin xyz="0 0 0.10" rpy="0 0 0"/>
         </collision>
-        <xacro:arm6_link xyz="0 0 0.10531595" rpy="0 0 0" />
     </link>
     <joint name="base_joint" type="fixed">

File: src/6dof_arm_description/urdf/properties.urdf.xacro (robot description, xacro)
@@ -22,5 +22,5 @@
         <color rgba="0.5372 0.8549 0.8274 1.0"/>
     </material>
-    <xacro:macro name="base_link" params="xyz rpy">
+    <xacro:macro name="base_inertia" params="xyz rpy">
         <inertial>
             <origin xyz="${xyz}" rpy="${rpy}" />
@@ -31,5 +31,5 @@
         </inertial>
     </xacro:macro>
-    <xacro:macro name="arm1_link" params="xyz rpy">
+    <xacro:macro name="arm1_inertia" params="xyz rpy">
         <inertial>
             <origin xyz="${xyz}" rpy="${rpy}" />
@@ -40,5 +40,5 @@
         </inertial>
     </xacro:macro>
-    <xacro:macro name="arm2_link" params="xyz rpy">
+    <xacro:macro name="arm2_inertia" params="xyz rpy">
         <inertial>
             <origin xyz="${xyz}" rpy="${rpy}" />
@@ -49,5 +49,5 @@
         </inertial>
     </xacro:macro>
-    <xacro:macro name="arm3_link" params="xyz rpy">
+    <xacro:macro name="arm3_inertia" params="xyz rpy">
         <inertial>
             <origin xyz="${xyz}" rpy="${rpy}" />
@@ -58,5 +58,5 @@
         </inertial>
     </xacro:macro>
-    <xacro:macro name="arm4_link" params="xyz rpy">
+    <xacro:macro name="arm4_inertia" params="xyz rpy">
         <inertial>
             <origin xyz="${xyz}" rpy="${rpy}" />
@@ -67,5 +67,5 @@
         </inertial>
     </xacro:macro>
-    <xacro:macro name="arm5_link" params="xyz rpy">
+    <xacro:macro name="arm5_inertia" params="xyz rpy">
         <inertial>
             <origin xyz="${xyz}" rpy="${rpy}" />
@@ -76,5 +76,5 @@
         </inertial>
     </xacro:macro>
-    <xacro:macro name="arm6_link" params="xyz rpy">
+    <xacro:macro name="arm6_inertia" params="xyz rpy">
         <inertial>
             <origin xyz="${xyz}" rpy="${rpy}" />

Commit message: Implementação de launch para o gazebo

File: src/6dof_arm_description/urdf/6dof_arm.urdf.xacro (robot description, xacro)
@@ -1,4 +1,5 @@
 <?xml version="1.0"?>
 <robot name="6dof_arm" xmlns:xacro="http://www.ros.org/wiki/xacro">
+    <xacro:include filename="mobile_base_gazebo.xacro"/>
     <xacro:include filename="properties.urdf.xacro"/>
     <xacro:include filename="mobile_base.urdf.xacro"/>

File: src/6dof_arm_description/urdf/mobile_base.urdf.xacro (robot description, xacro)
@@ -1,5 +1,4 @@
 <?xml version="1.0"?>
 <robot xmlns:xacro="http://www.ros.org/wiki/xacro">
-    <link name="base_footprint"/>
     <link name="base_link">
         <visual>
@@ -42,5 +41,5 @@
             <material name="yellow"/>
         </visual>
-        <xacro:arm2_inertia xyz="-0.00008884 0 0.47500021" rpy="0 0 -${pi/2.0}" />
+        <xacro:arm2_inertia xyz="-0.00008884 0 0.47100021" rpy="0 0 -${pi/2.0}" />
         <collision>
             <geometry>
@@ -114,44 +113,51 @@
         </collision>
     </link>
-    <joint name="base_joint" type="fixed">
-        <parent link="base_footprint" />
-        <child link="base_link" />
-        <origin xyz ="0 0 0" rpy="0 0 0" />
+    <link name="world"/>
+    <joint name="world_base_joint" type="fixed">
+        <origin xyz="0 0 0" rpy="0 0 0"/>
+        <parent link="world"/>
+        <child link="base_link"/>
     </joint>
-    <joint name="base_arm1_joint" type="continuous">
+    <joint name="base_arm1_joint" type="revolute">
         <parent link="base_link" />
         <child link="arm1_link" />
         <origin xyz ="0 0 0.07" rpy="0 0 0" />
         <axis xyz="0 0 1" />
+        <limit lower="-${pi}" upper="${pi}" effort="10" velocity="1.0"/>
     </joint>
-    <joint name="arm1_arm2_joint" type="continuous">
+    <joint name="arm1_arm2_joint" type="revolute">
         <parent link="arm1_link" />
         <child link="arm2_link" />
         <origin xyz ="0 -0.20 0.20" rpy="0 0 0" />
         <axis xyz="0 1 0" />
+        <limit lower="-${pi}" upper="${pi}" effort="100" velocity="1.0"/>
     </joint>
-    <joint name="arm2_arm3_joint" type="continuous">
+    <joint name="arm2_arm3_joint" type="revolute">
         <parent link="arm2_link" />
         <child link="arm3_link" />
         <origin xyz ="0 0.20 0.95" rpy="0 0 0" />
         <axis xyz="0 1 0" />
+        <limit lower="-${pi}" upper="${pi}" effort="10" velocity="1.0"/>
     </joint>
-    <joint name="arm3_arm4_joint" type="continuous">
+    <joint name="arm3_arm4_joint" type="revolute">
         <parent link="arm3_link" />
         <child link="arm4_link" />
         <origin xyz ="0.65 -0.20 0" rpy="0 -${pi/2} 0" />
         <axis xyz="0 1 0" />
+        <limit lower="-${pi}" upper="${pi}" effort="10" velocity="1.0"/>
     </joint>
-    <joint name="arm4_arm5_joint" type="continuous">
+    <joint name="arm4_arm5_joint" type="revolute">
         <parent link="arm4_link" />
         <child link="arm5_link" />
         <origin xyz ="0 0 -0.20" rpy="0 0 ${pi}" />
         <axis xyz="0 0 1" />
+        <limit lower="-${pi}" upper="${pi}" effort="10" velocity="1.0"/>
     </joint>
-    <joint name="arm5_arm6_joint" type="continuous">
+    <joint name="arm5_arm6_joint" type="revolute">
         <parent link="arm5_link" />
         <child link="arm6_link" />
         <origin xyz ="0.10 0 -0.1" rpy="0 ${pi/2} 0" />
         <axis xyz="0 0 1" />
+        <limit lower="-${pi}" upper="${pi}" effort="10" velocity="1.0"/>
     </joint>
 </robot>
