Commit message: Implementação de controle do robô

File: src/6dof_arm_description/urdf/6dof_arm.urdf.xacro (robot description, xacro)
@@ -1,4 +1,5 @@
 <?xml version="1.0"?>
 <robot name="6dof_arm" xmlns:xacro="http://www.ros.org/wiki/xacro">
+    <xacro:include filename="ros2_control.xacro"/>
     <xacro:include filename="mobile_base_gazebo.xacro"/>
     <xacro:include filename="properties.urdf.xacro"/>

File: src/6dof_arm_description/urdf/mobile_base.urdf.xacro (robot description, xacro)
@@ -124,5 +124,5 @@
         <origin xyz ="0 0 0.07" rpy="0 0 0" />
         <axis xyz="0 0 1" />
-        <limit lower="-${pi}" upper="${pi}" effort="10" velocity="1.0"/>
+        <limit lower="0" upper="${pi}" effort="10" velocity="1.0"/>
     </joint>
     <joint name="arm1_arm2_joint" type="revolute">
@@ -131,5 +131,5 @@
         <origin xyz ="0 -0.20 0.20" rpy="0 0 0" />
         <axis xyz="0 1 0" />
-        <limit lower="-${pi}" upper="${pi}" effort="100" velocity="1.0"/>
+        <limit lower="0" upper="${pi}" effort="100" velocity="1.0"/>
     </joint>
     <joint name="arm2_arm3_joint" type="revolute">
@@ -138,5 +138,5 @@
         <origin xyz ="0 0.20 0.95" rpy="0 0 0" />
         <axis xyz="0 1 0" />
-        <limit lower="-${pi}" upper="${pi}" effort="10" velocity="1.0"/>
+        <limit lower="0" upper="${pi}" effort="10" velocity="1.0"/>
     </joint>
     <joint name="arm3_arm4_joint" type="revolute">
@@ -145,5 +145,5 @@
         <origin xyz ="0.65 -0.20 0" rpy="0 -${pi/2} 0" />
         <axis xyz="0 1 0" />
-        <limit lower="-${pi}" upper="${pi}" effort="10" velocity="1.0"/>
+        <limit lower="0" upper="${pi}" effort="10" velocity="1.0"/>
     </joint>
     <joint name="arm4_arm5_joint" type="revolute">
@@ -152,5 +152,5 @@
         <origin xyz ="0 0 -0.20" rpy="0 0 ${pi}" />
         <axis xyz="0 0 1" />
-        <limit lower="-${pi}" upper="${pi}" effort="10" velocity="1.0"/>
+        <limit lower="0" upper="${pi}" effort="10" velocity="1.0"/>
     </joint>
     <joint name="arm5_arm6_joint" type="revolute">
@@ -159,5 +159,5 @@
         <origin xyz ="0.10 0 -0.1" rpy="0 ${pi/2} 0" />
         <axis xyz="0 0 1" />
-        <limit lower="-${pi}" upper="${pi}" effort="10" velocity="1.0"/>
+        <limit lower="0" upper="${pi}" effort="10" velocity="1.0"/>
     </joint>
 </robot>

Commit message: Implementação de sensor Lidar

File: src/6dof_arm_description/urdf/6dof_arm.urdf.xacro (robot description, xacro)
@@ -2,6 +2,6 @@
 <robot name="6dof_arm" xmlns:xacro="http://www.ros.org/wiki/xacro">
     <xacro:include filename="ros2_control.xacro"/>
-    <xacro:include filename="mobile_base_gazebo.xacro"/>
-    <xacro:include filename="properties.urdf.xacro"/>
+    <xacro:include filename="6dof_arm_properties.urdf.xacro"/>
     <xacro:include filename="mobile_base.urdf.xacro"/>
+    <xacro:include filename="lidar_sensor.urdf.xacro"/>
 </robot>

File: src/6dof_arm_description/urdf/6dof_arm_properties.urdf.xacro (robot description, xacro)
@@ -85,3 +85,27 @@
         </inertial>
     </xacro:macro>
+    <xacro:macro name="gazebo_material" params="link ambient">
+        <gazebo reference="${link}">
+            <selfCollide>true</selfCollide>
+            <visual>
+                <material>
+                    <ambient>${ambient}</ambient>
+                    <diffuse>0.9 0.6 0.45 1</diffuse>
+                    <specular>0.95 0.95 0.95 1</specular>
+                    <emissive>0 0 0 0</emissive>
+                </material>
+                <mu1>0.2</mu1>
+                <mu2>0.2</mu2>
+                <self_collide>true</self_collide>
+                <gravity>true</gravity>
+            </visual>
+        </gazebo>
+    </xacro:macro>
+    <xacro:gazebo_material link="base_link" ambient="0.5 0.5 0.5" />
+    <xacro:gazebo_material link="arm1_link" ambient="0.8754 0.4471 0.3176" />
+    <xacro:gazebo_material link="arm2_link" ambient="1 0.7569 0.0549" />
+    <xacro:gazebo_material link="arm3_link" ambient="0.6824 0.3333 0.7373" />
+    <xacro:gazebo_material link="arm4_link" ambient="0.3725 0.6549 0.2392" />
+    <xacro:gazebo_material link="arm5_link" ambient="0.3686 0.2509 0.6431" />
+    <xacro:gazebo_material link="arm6_link" ambient="0.5372 0.8549 0.8274" />
 </robot>
