Commit message: Adição dos grippers

File: src/6dof_arm_description/urdf/6dof_arm_properties.urdf.xacro (robot description, xacro)
@@ -85,4 +85,13 @@
         </inertial>
     </xacro:macro>
+    <xacro:macro name="gripper_inertia" params="xyz rpy">
+        <inertial>
+            <origin xyz="${xyz}" rpy="${rpy}" />
+            <mass value="0.23129816" />
+            <inertia ixx="0.00058838" ixy="-0.00002395" ixz="0"
+                     iyy="0.00007385"  iyz="0"
+                     izz="0.00065355" />
+        </inertial>
+    </xacro:macro>
     <xacro:macro name="gazebo_material" params="link ambient">
         <gazebo reference="${link}">
@@ -109,3 +118,5 @@
     <xacro:gazebo_material link="arm5_link" ambient="0.3686 0.2509 0.6431" />
     <xacro:gazebo_material link="arm6_link" ambient="0.5372 0.8549 0.8274" />
+    <xacro:gazebo_material link="gripper1_link" ambient="0.5 0.5 0.5" />
+    <xacro:gazebo_material link="gripper2_link" ambient="0.5 0.5 0.5" />
 </robot>

File: src/6dof_arm_description/urdf/mobile_base.urdf.xacro (robot description, xacro)
@@ -111,4 +111,36 @@
             </geometry>
             <origin xyz="0 0 0.10" rpy="0 0 0"/>
+        </collision>
+    </link>
+    <link name="gripper1_link">
+        <visual>
+            <geometry>
+                <mesh filename="package://6dof_arm_description/meshes/6dof_arm/gripper.stl" scale="1 1 1"/>
+            </geometry>
+            <origin xyz="0 0 0" rpy="0 ${pi/2} 0"/>
+            <material name="light_black"/>
+        </visual>
+        <xacro:gripper_inertia xyz="-0.0075 0.090250025 0.027995235" rpy="0 0 0" />
+        <collision>
+            <geometry>
+                <box size="0.015 0.16050005 0.07295455" />
+            </geometry>
+            <origin xyz="-0.0075 0.090250025 0.027995235" rpy="0 0 0"/>
+        </collision>
+    </link>
+    <link name="gripper2_link">
+        <visual>
+            <geometry>
+                <mesh filename="package://6dof_arm_description/meshes/6dof_arm/gripper.stl" scale="1 1 1"/>
+            </geometry>
+            <origin xyz="0 0 0" rpy="0 ${pi/2} 0"/>
+            <material name="light_black"/>
+        </visual>
+        <xacro:gripper_inertia xyz="-0.0075 0.090250025 0.027995235" rpy="0 0 0" />
+        <collision>
+            <geometry>
+                <box size="0.015 0.16050005 0.07295455" />
+            </geometry>
+            <origin xyz="-0.0075 0.090250025 0.027995235" rpy="0 0 0"/>
         </collision>
     </link>
@@ -161,3 +193,17 @@
         <limit lower="0" upper="${pi}" effort="10" velocity="1.0"/>
     </joint>
+    <joint name="arm6_gripper1_joint" type="revolute">
+        <parent link="arm6_link" />
+        <child link="gripper1_link" />
+        <origin xyz ="-0.0075 0.025 0.245" rpy="0 ${pi} 0" />
+        <axis xyz="1 0 0" />
+        <limit lower="${-pi/4}" upper="${-pi/2}" effort="10" velocity="1.0"/>
+    </joint>
+    <joint name="arm6_gripper2_joint" type="revolute">
+        <parent link="arm6_link" />
+        <child link="gripper2_link" />
+        <origin xyz ="0.0075 -0.025 0.245" rpy="0 0 0" />
+        <axis xyz="1 0 0" />
+        <limit lower="${pi/2}" upper="${3/4*pi}" effort="10" velocity="1.0"/>
+    </joint>
 </robot>

File: src/6dof_arm_description/urdf/ros2_control.xacro (robot description, xacro)
@@ -77,4 +77,28 @@
             <state_interface name="position" />
         </joint>
+        <joint name="arm6_gripper1_joint">
+            <command_interface name="position">
+                <param name="min">${-pi/4}</param>
+                <param name="max">${-pi/2}</param>
+            </command_interface>
+            <state_interface name="position">
+                <param name="initial_value">0.0</param>
+            </state_interface>
+            <state_interface name="velocity" />
+            <state_interface name="effort" />
+            <state_interface name="position" />
+        </joint>
+        <joint name="arm6_gripper2_joint">
+            <command_interface name="position">
+                <param name="min">${pi/2}</param>
+                <param name="max">${3/4*pi}</param>
+            </command_interface>
+            <state_interface name="position">
+                <param name="initial_value">0.0</param>
+            </state_interface>
+            <state_interface name="velocity" />
+            <state_interface name="effort" />
+            <state_interface name="position" />
+        </joint>
     </ros2_control>
     <gazebo>
