Commit message: Adição de sensor de contato e correção de ângulos mínimo e máximo dos links do braço

File: src/sixdof_arm_description/urdf/mobile_base.urdf.xacro (robot description, xacro)
@@ -1,4 +1,7 @@
 <?xml version="1.0"?>
-<robot xmlns:xacro="http://www.ros.org/wiki/xacro">
+<robot name="sixdof_arm" xmlns:xacro="http://www.ros.org/wiki/xacro">
+<!-- =================================================================================== -->
+<!-- |                                    LINKS                                        | -->
+<!-- =================================================================================== -->
     <link name="base_link">
         <visual>
@@ -26,5 +29,5 @@
         </visual>
         <xacro:arm1_inertia xyz="0 -0.00016159 0.14671717" rpy="0 0 0" />
-        <collision>
+        <collision name="arm1_link_collision">
             <geometry>
                 <box size="0.15 0.20 0.275" />
@@ -42,5 +45,5 @@
         </visual>
         <xacro:arm2_inertia xyz="-0.00008884 0 0.47100021" rpy="0 0 -${pi/2.0}" />
-        <collision>
+        <collision name="arm2_link_collision">
             <geometry>
                 <box size="0.15 0.20 1.10" />
@@ -58,5 +61,5 @@
         </visual>
         <xacro:arm3_inertia xyz="0.325 0 -0.00011793" rpy="0 ${pi/2} 0" />
-        <collision>
+        <collision name="arm3_link_collision">
             <geometry>
                 <box size="0.15 0.20 0.80" />
@@ -74,5 +77,5 @@
         </visual>
         <xacro:arm4_inertia xyz="0 0.0010614 -0.05328286" rpy="${pi} 0 0" />
-        <collision>
+        <collision name="arm4_link_collision">
             <geometry>
                 <box size="0.15 0.20 0.275" />
@@ -90,5 +93,5 @@
         </visual>
         <xacro:arm5_inertia xyz="-0.0002301 0 -0.08772699" rpy="${pi} 0 ${pi}" />
-        <collision>
+        <collision name="arm5_link_collision">
             <geometry>
                 <box size="0.20 0.15 0.175" />
@@ -106,5 +109,5 @@
         </visual>
         <xacro:arm6_inertia xyz="0 0 0.10531595" rpy="0 0 0" />
-        <collision>
+        <collision name="arm6_link_collision">
             <geometry>
                 <box size="0.15 0.15 0.20" />
@@ -122,5 +125,5 @@
         </visual>
         <xacro:gripper_inertia xyz="-0.0075 0.090250025 0.027995235" rpy="0 0 0" />
-        <collision>
+        <collision name="gripper1_link_collision">
             <geometry>
                 <box size="0.015 0.16050005 0.07295455" />
@@ -138,5 +141,5 @@
         </visual>
         <xacro:gripper_inertia xyz="-0.0075 0.090250025 0.027995235" rpy="0 0 0" />
-        <collision>
+        <collision name="gripper2_link_collision">
             <geometry>
                 <box size="0.015 0.16050005 0.07295455" />
@@ -146,4 +149,7 @@
     </link>
     <link name="world"/>
+<!-- =================================================================================== -->
+<!-- |                                    JOINTS                                       | -->
+<!-- =================================================================================== -->
     <joint name="world_base_joint" type="fixed">
         <origin xyz="0 0 0" rpy="0 0 0"/>
@@ -156,5 +162,5 @@
         <origin xyz ="0 0 0.07" rpy="0 0 0" />
         <axis xyz="0 0 1" />
-        <limit lower="0" upper="${pi}" effort="10" velocity="1.0"/>
+        <limit lower="${-pi/2}" upper="${pi/2}" effort="10" velocity="1.0"/>
     </joint>
     <joint name="arm1_arm2_joint" type="revolute">
@@ -163,5 +169,5 @@
         <origin xyz ="0 -0.20 0.20" rpy="0 0 0" />
         <axis xyz="0 1 0" />
-        <limit lower="0" upper="${pi}" effort="100" velocity="1.0"/>
+        <limit lower="${-pi/2}" upper="${pi/2}" effort="10" velocity="1.0"/>
     </joint>
     <joint name="arm2_arm3_joint" type="revolute">
@@ -170,5 +176,5 @@
         <origin xyz ="0 0.20 0.95" rpy="0 0 0" />
         <axis xyz="0 1 0" />
-        <limit lower="0" upper="${pi}" effort="10" velocity="1.0"/>
+        <limit lower="${-pi/2}" upper="${pi/2}" effort="10" velocity="1.0"/>
     </joint>
     <joint name="arm3_arm4_joint" type="revolute">
@@ -177,5 +183,5 @@
         <origin xyz ="0.65 -0.20 0" rpy="0 -${pi/2} 0" />
         <axis xyz="0 1 0" />
-        <limit lower="0" upper="${pi}" effort="10" velocity="1.0"/>
+        <limit lower="${-pi/2}" upper="${pi/2}" effort="10" velocity="1.0"/>
     </joint>
     <joint name="arm4_arm5_joint" type="revolute">
@@ -184,5 +190,5 @@
         <origin xyz ="0 0 -0.20" rpy="0 0 ${pi}" />
         <axis xyz="0 0 1" />
-        <limit lower="0" upper="${pi}" effort="10" velocity="1.0"/>
+        <limit lower="${-pi/2}" upper="${pi/2}" effort="10" velocity="1.0"/>
     </joint>
     <joint name="arm5_arm6_joint" type="revolute">
@@ -191,5 +197,5 @@
         <origin xyz ="0.10 0 -0.1" rpy="0 ${pi/2} 0" />
         <axis xyz="0 0 1" />
-        <limit lower="0" upper="${pi}" effort="10" velocity="1.0"/>
+        <limit lower="${-pi/2}" upper="${pi/2}" effort="10" velocity="1.0"/>
     </joint>
     <joint name="arm6_gripper1_joint" type="revolute">
@@ -207,51 +213,25 @@
         <limit lower="${pi/2}" upper="${3/4*pi}" effort="10" velocity="1.0"/>
     </joint>
-    <transmission name="transmission_base_arm1">
-        <type>transmission_interface/SimpleTransmission</type>
-        <joint name="base_arm1_joint">
-            <hardwareInterface>velocity</hardwareInterface>
-        </joint>
-    </transmission>
-    <transmission name="transmission_arm1_arm2_joint">
-        <type>transmission_interface/SimpleTransmission</type>
-        <joint name="arm1_arm2_joint">
-            <hardwareInterface>velocity</hardwareInterface>
-        </joint>
-    </transmission>
-    <transmission name="transmission_arm2_arm3_joint">
-        <type>transmission_interface/SimpleTransmission</type>
-        <joint name="arm2_arm3_joint">
-            <hardwareInterface>velocity</hardwareInterface>
-        </joint>
-    </transmission>
-    <transmission name="transmission_arm3_arm4_joint">
-        <type>transmission_interface/SimpleTransmission</type>
-        <joint name="arm3_arm4_joint">
-            <hardwareInterface>velocity</hardwareInterface>
-        </joint>
-    </transmission>
-    <transmission name="transmission_arm4_arm5_joint">
-        <type>transmission_interface/SimpleTransmission</type>
-        <joint name="arm4_arm5_joint">
-            <hardwareInterface>velocity</hardwareInterface>
-        </joint>
-    </transmission>
-    <transmission name="transmission_arm5_arm6_joint">
-        <type>transmission_interface/SimpleTransmission</type>
-        <joint name="arm5_arm6_joint">
-            <hardwareInterface>velocity</hardwareInterface>
-        </joint>
-    </transmission>
-    <transmission name="transmission_arm6_gripper1_joint">
-        <type>transmission_interface/SimpleTransmission</type>
-        <joint name="arm6_gripper1_joint">
-            <hardwareInterface>velocity</hardwareInterface>
-        </joint>
-    </transmission>
-    <transmission name="transmission_arm6_gripper2_joint">
-        <type>transmission_interface/SimpleTransmission</type>
-        <joint name="arm6_gripper2_joint">
-            <hardwareInterface>velocity</hardwareInterface>
-        </joint>
-    </transmission>
+<!-- =================================================================================== -->
+<!-- |                               TRANSMISSION                                       | -->
+<!-- =================================================================================== -->
+    <xacro:transmission joint_name="base_arm1_joint" />
+    <xacro:transmission joint_name="arm1_arm2_joint" />
+    <xacro:transmission joint_name="arm2_arm3_joint" />
+    <xacro:transmission joint_name="arm3_arm4_joint" />
+    <xacro:transmission joint_name="arm4_arm5_joint" />
+    <xacro:transmission joint_name="arm5_arm6_joint" />
+    <xacro:transmission joint_name="arm6_gripper1_joint" />
+    <xacro:transmission joint_name="arm6_gripper2_joint" />
+<!-- =================================================================================== -->
+<!-- |                               CONTACT SENSOR                                    | -->
+<!-- =================================================================================== -->
+    <xacro:contact_sensor reference="arm1_link" />
+    <xacro:contact_sensor reference="arm2_link" />
+    <xacro:contact_sensor reference="arm3_link" />
+    <xacro:contact_sensor reference="arm4_link" />
+    <xacro:contact_sensor reference="arm5_link" />
+    <xacro:contact_sensor reference="arm6_link" />
+    <xacro:contact_sensor reference="gripper1_link" />
+    <xacro:contact_sensor reference="gripper2_link" />
 </robot>

File: src/sixdof_arm_description/urdf/ros2_control.xacro (robot description, xacro)
@@ -7,6 +7,6 @@
         <joint name="base_arm1_joint">
             <command_interface name="position">
-                <param name="min">0</param>
-                <param name="max">${pi}</param>
+                <param name="min">${-pi/2}</param>
+                <param name="max">${pi/2}</param>
             </command_interface>
             <command_interface name="velocity">
@@ -23,6 +23,6 @@
         <joint name="arm1_arm2_joint">
             <command_interface name="position">
-                <param name="min">0</param>
-                <param name="max">${pi}</param>
+                <param name="min">${-pi/2}</param>
+                <param name="max">${pi/2}</param>
             </command_interface>
             <command_interface name="velocity">
@@ -39,6 +39,6 @@
         <joint name="arm2_arm3_joint">
             <command_interface name="position">
-                <param name="min">0</param>
-                <param name="max">${pi}</param>
+                <param name="min">${-pi/2}</param>
+                <param name="max">${pi/2}</param>
             </command_interface>
             <command_interface name="velocity">
@@ -55,6 +55,6 @@
         <joint name="arm3_arm4_joint">
             <command_interface name="position">
-                <param name="min">0</param>
-                <param name="max">${pi}</param>
+                <param name="min">${-pi/2}</param>
+                <param name="max">${pi/2}</param>
             </command_interface>
             <command_interface name="velocity">
@@ -71,6 +71,6 @@
         <joint name="arm4_arm5_joint">
             <command_interface name="position">
-                <param name="min">0</param>
-                <param name="max">${pi}</param>
+                <param name="min">${-pi/2}</param>
+                <param name="max">${pi/2}</param>
             </command_interface>
             <command_interface name="velocity">
@@ -87,6 +87,6 @@
         <joint name="arm5_arm6_joint">
             <command_interface name="position">
-                <param name="min">0</param>
-                <param name="max">${pi}</param>
+                <param name="min">${-pi/2}</param>
+                <param name="max">${pi/2}</param>
             </command_interface>
             <command_interface name="velocity">

File: src/sixdof_arm_description/urdf/sixdof_arm_properties.urdf.xacro (robot description, xacro)
@@ -120,3 +120,30 @@
     <xacro:gazebo_material link="gripper1_link" ambient="0.5 0.5 0.5" />
     <xacro:gazebo_material link="gripper2_link" ambient="0.5 0.5 0.5" />
+    <xacro:macro name="contact_sensor" params="reference">
+        <gazebo reference="${reference}">
+        <sensor name="${reference}_bumper" type="contact">
+            <always_on>true</always_on>
+            <update_rate>50</update_rate>
+            <contact>
+                <collision>${reference}_collision_collision</collision>
+            </contact>
+            <plugin name="${reference}_contact_plugin" filename="libgazebo_ros_bumper.so">
+                <ros>
+                    <remapping>bumper_states:=${reference}_bumper</remapping>
+                </ros>
+                <alwaysOn>true</alwaysOn>
+                <update_rate>50.0</update_rate>
+                <frameName>${reference}</frameName>
+            </plugin>
+        </sensor>
+    </gazebo>
+    </xacro:macro>
+    <xacro:macro name="transmission" params="joint_name">
+        <transmission name="transmission_${joint_name}">
+            <type>transmission_interface/SimpleTransmission</type>
+            <joint name="joint_name">
+                <hardwareInterface>velocity</hardwareInterface>
+            </joint>
+        </transmission>
+    </xacro:macro>
 </robot>
